Commit message: Added gazebo plugin

File: description/robot_core.xacro (robot description, xacro)
@@ -1,21 +1,21 @@
 <?xml version="1.0"?>
-<robot xmlns:xacro="http://www.ros.org/wiki/xacro" >
-    <xacro:include filename="inertial_macros.xacro"/>
+<robot xmlns:xacro="http://www.ros.org/wiki/xacro"  >
+    <xacro:include filename="inertial_macro.xacro"/>
     <material name="white">
         <color rgba="1 1 1 1" />
     </material>
     <material name="orange">
-        <color rgba="1 0.3 0.1 1"/>
+        <color rgba="1 0.3 0.1 1" />
     </material>
     <material name="blue">
-        <color rgba="0.2 0.2 1 1"/>
+        <color rgba="0.2 0.2 1 1" />
     </material>
     <material name="black">
-        <color rgba="0 0 0 1"/>
+        <color rgba="0 0 0 1" />
     </material>
-    <!-- BASE LINK -->
+    <!--BASE LINK-->
     <link name="base_link">
     </link>
-    <!-- CHASSIS LINK -->
+    <!--CHASSIS LINK-->
     <joint name="chassis_joint" type="fixed">
         <parent link="base_link"/>
@@ -31,5 +31,5 @@
             <material name="white"/>
         </visual>
-        <collision>
+      <collision>
             <origin xyz="0.15 0 0.075"/>
             <geometry>
@@ -41,9 +41,9 @@
         </xacro:inertial_box>
     </link>
-    <!-- LEFT WHEEL LINK -->
-    <joint name="left_wheel_joint" type="continuous">
+    <!--LEFT WHEEL LINK-->
+    <joint name="left_wheel_join" type="continuous">
         <parent link="base_link"/>
         <child link="left_wheel"/>
-        <origin xyz="0 0.175 0" rpy="-${pi/2} 0 0" />
+        <origin xyz="0 0.175 0" rpy="-${pi/2} 0 0"/>
         <axis xyz="0 0 1"/>
     </joint>
@@ -64,9 +64,9 @@
         </xacro:inertial_cylinder>
     </link>
-    <!-- RIGHT WHEEL LINK -->
-    <joint name="right_wheel_joint" type="continuous">
+    <!--RIGHT WHEEL LINK-->
+    <joint name="right_wheel_join" type="continuous">
         <parent link="base_link"/>
         <child link="right_wheel"/>
-        <origin xyz="0 -0.175 0" rpy="${pi/2} 0 0" />
+        <origin xyz="0 -0.175 0" rpy="${pi/2} 0 0"/>
         <axis xyz="0 0 -1"/>
     </joint>
@@ -87,5 +87,5 @@
         </xacro:inertial_cylinder>
     </link>
-    <!-- CASTER WHEEL LINK -->
+    <!--CASTER WHEEL LINK-->
     <joint name="caster_wheel_joint" type="fixed">
         <parent link="chassis"/>
@@ -106,5 +106,5 @@
         </collision>
         <xacro:inertial_sphere mass="0.1" radius="0.05">
-            <origin xyz="0 0 0" rpy="0 0 0"/>
+        <origin xyz="0 0 0" rpy="0 0 0"/>
         </xacro:inertial_sphere>
     </link>
